File: LoRa_Board_STM32WL55JCI6.kicad_sch (KiCad schematic)
At the start: 123 parts, among them J1 LPUART1_Headers, J10 Power Select Jumpers, J11 Debug_Pins, J13 SMA PCB END LAUNCH JACK ROUND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, J14 USB_B_Micro, J15 BOOT0_Jumper, J2 I2C1_Headers, J3 Power Pins, J4 Pin_Headers, J5 SPI1_Headers, J6 Power Select Jumpers, J7 Coin Battery Jumper, J8 BOOT0_Jumper, J9 User Button Jumper, U1 STM32WL55CCU6, U4 FT230XS, U5 USBLC6-2SC6, U6 BGS12WN6E6327, U7 STM32WL55JCI6, U8 STM32WL55JCIx, Y1 ABM3B-32.000MHZ-8-R30-B1U-T, Y2 Clock_ECS-327MVATX-7-CN-TR, Y3 ABM3B-32.000MHZ-8-R30-B1U-T, Y6 Clock_ECS-327MVATX-7-CN-TR

Commit message: Update
Parts:
- removed C1, C4, C43, C46, C48, C6: 33p_GJM0335C1E330JB01D_MURATA, Capacitor_SMD:C_0805_2012Metric_Pad1.18x1.45mm_HandSolder, symbol Device:C
- removed C10, C60: 10n, Capacitor_SMD:C_0805_2012Metric_Pad1.18x1.45mm_HandSolder, symbol Device:C
- removed C11, C13, C2, C44, C49, C51, C53, C55, C59, C7, C9: 100n, Capacitor_SMD:C_0805_2012Metric_Pad1.18x1.45mm_HandSolder, symbol Device:C
- removed C12, C54: 470n, Capacitor_SMD:C_0805_2012Metric_Pad1.18x1.45mm_HandSolder, symbol Device:C
- removed C14, C56: 1u, Capacitor_SMD:C_0805_2012Metric_Pad1.18x1.45mm_HandSolder, symbol Device:C
- removed C15, C57: 1uF, Capacitor_SMD:C_0805_2012Metric_Pad1.18x1.45mm_HandSolder, symbol Device:C
- removed C17, C3, C45, C50, C58, C8: 4u7, Capacitor_SMD:C_0805_2012Metric_Pad1.18x1.45mm_HandSolder, symbol Device:C
- removed C47, C5: 100n_FCC0402KRX7R7BB104, Capacitor_SMD:C_0805_2012Metric_Pad1.18x1.45mm_HandSolder, symbol Device:C
- removed FB3: ILB1206ER700V_1206, Capacitor_SMD:C_1206_3216Metric_Pad1.33x1.80mm_HandSolder, symbol Device:FerriteBead
- removed J15, J8: BOOT0_Jumper, Connector_PinHeader_2.54mm:PinHeader_1x03_P2.54mm_Vertical, symbol Connector:Conn_01x03_Pin
- removed L1, L8: 15u_MLZ2012M150W_TDK, Inductor_SMD:L_0805_2012Metric_Pad1.15x1.40mm_HandSolder, symbol Device:L
- removed R10, R16: 1k, Resistor_SMD:R_0805_2012Metric_Pad1.20x1.40mm_HandSolder, symbol Device:R
- removed R18, R9: 10R, Resistor_SMD:R_0805_2012Metric_Pad1.20x1.40mm_HandSolder, symbol Device:R
- removed U1: STM32WL55CCU6, Package_DFN_QFN:QFN-48-1EP_7x7mm_P0.5mm_EP5.6x5.6mm, symbol MCU_ST_STM32WL:STM32WL55CCUx
- removed U2, U9: ~, Personal_Project:Button_KMR231GLFS, symbol Personal_Projects:Button_KMR231GLFS
- removed U7: STM32WL55JCI6, Package_BGA:ST_UFBGA-73_5x5mm_Layout9x9_P0.5mm, symbol MCU_ST_STM32WL:STM32WL55JCIx
- removed U8: STM32WL55JCIx, Package_BGA:ST_UFBGA-73_5x5mm_Layout9x9_P0.5mm, symbol MCU_ST_STM32WL:STM32WL55JCIx
- removed Y1, Y3: ABM3B-32.000MHZ-8-R30-B1U-T, Personal_Project:XTAL_ABM3B-32.000MHZ-10-R30-B1U-T, symbol Personal_Projects:ABM3B-32.000MHZ-10-R30-B1U-T
- removed Y2, Y6: Clock_ECS-327MVATX-7-CN-TR, Personal_Project:Clock_ECS327MVATX7CNTR, symbol Personal_Projects:Clock_ECS-327MVATX-7-CN-TR
- added C52, C63, C65: 33p_GJM0335C1E330JB01D_MURATA, Capacitor_SMD:C_0805_2012Metric_Pad1.18x1.45mm_HandSolder, symbol Device:C
- added C61, C66, C68, C69, C70, C73: 100n, Capacitor_SMD:C_0805_2012Metric_Pad1.18x1.45mm_HandSolder, symbol Device:C
- added C62, C67, C76: 4u7, Capacitor_SMD:C_0805_2012Metric_Pad1.18x1.45mm_HandSolder, symbol Device:C
- added C64: 100n_FCC0402KRX7R7BB104, Capacitor_SMD:C_0805_2012Metric_Pad1.18x1.45mm_HandSolder, symbol Device:C
- added C71: 1u, Capacitor_SMD:C_0805_2012Metric_Pad1.18x1.45mm_HandSolder, symbol Device:C
- added C72: 470n, Capacitor_SMD:C_0805_2012Metric_Pad1.18x1.45mm_HandSolder, symbol Device:C
- added C74: 1uF, Capacitor_SMD:C_0805_2012Metric_Pad1.18x1.45mm_HandSolder, symbol Device:C
- added C75: 10n, Capacitor_SMD:C_0805_2012Metric_Pad1.18x1.45mm_HandSolder, symbol Device:C
- added J16: BOOT0_Jumper, Connector_PinHeader_2.54mm:PinHeader_1x03_P2.54mm_Vertical, symbol Connector:Conn_01x03_Pin
- added J8: Pin_Headers_1, Connector_PinHeader_2.54mm:PinHeader_2x07_P2.54mm_Vertical, symbol Connector_Generic:Conn_02x07_Odd_Even
- added L9: 15u_MLZ2012M150W_TDK, Inductor_SMD:L_0805_2012Metric_Pad1.15x1.40mm_HandSolder, symbol Device:L
- added R17: 10R, Resistor_SMD:R_0805_2012Metric_Pad1.20x1.40mm_HandSolder, symbol Device:R
- added R19: 1k, Resistor_SMD:R_0805_2012Metric_Pad1.20x1.40mm_HandSolder, symbol Device:R
- added U10: STM32WL55JCI6, Package_BGA:ST_UFBGA-73_5x5mm_Layout9x9_P0.5mm, symbol MCU_ST_STM32WL:STM32WL55JCIx
- added U11: ~, Personal_Project:Button_KMR231GLFS, symbol Personal_Projects:Button_KMR231GLFS
- added Y4: ABM3B-32.000MHZ-8-R30-B1U-T, Personal_Project:XTAL_ABM3B-32.000MHZ-10-R30-B1U-T, symbol Personal_Projects:ABM3B-32.000MHZ-10-R30-B1U-T
- added Y5: Clock_ECS-327MVATX-7-CN-TR, Personal_Project:Clock_ECS327MVATX7CNTR, symbol Personal_Projects:Clock_ECS-327MVATX-7-CN-TR
- FB1: value ILB1206ER700V_1206 -> BLM21PG601SN1D_0805; footprint Capacitor_SMD:C_1206_3216Metric_Pad1.33x1.80mm_HandSolder -> Capacitor_SMD:C_0805_2012Metric_Pad1.18x1.45mm_HandSolder
- J4: value Pin_Headers -> Pin_Headers_2
Connections:
- net +3.3V: now also C52.1, C61.1, C62.1, C64.1, C65.1, C68.1, C69.1, C70.1, C71.1, C73.1, C75.2, C76.1, J16.1 (Pin_1), U10.A2 (VDDSMPS), U10.A7 (VDD), U10.E2 (VDD), U10.E8 (VDDRF), U10.E9 (VDD), U10.H5 (VDD), U10.H8 (VDDPA), Y5.4 (VDD)
- net +3.3VA: now also C66.1, C67.1, U10.A5 (VDDA), U10.B5 (VREF+)
- net BOOT0: now also R19.2, U10.J5 (PH3)
- net BOOT0J: now also J16.2 (Pin_2), R19.1
- net GND: now also C52.2, C61.2, C62.2, C63.2, C64.2, C65.2, C66.2, C67.2, C68.2, C69.2, C70.2, C71.2, C72.2, C73.2, C74.1, C75.1, C76.2, J16.3 (Pin_3), J8.14 (Pin_14), U10.A1 (VSSSMPS), U10.B7 (VSS), U10.D9 (VSS), U10.E3 (VSS), U10.G5 (VSS), U10.G6 (VSSRF), U10.G7 (VSSRF), U10.G8 (VSSRF), U10.H6 (VSSRF), U11.3, U11.4, U11.5 (GND), Y4.2, Y4.4, Y5.2 (GND); no longer J4.12 (Pin_12)
- net NRST: now also C74.2, U10.F5 (NRST), U11.1, U11.2
- net PA0: now also J8.1 (Pin_1), U10.D6 (PA0); no longer J4.1 (Pin_1)
- net PA10_USART1_RX: now also U10.C8 (PA10)
- net PA11_USART1_CTS: now also U10.B9 (PA11)
- net PA12_USART1_RTS: now also U10.A9 (PA12)
- net PA13_SWDIO: now also U10.B8 (PA13)
- net PA14_SWCLK: now also U10.A4 (PA14)
- net PA15: now also J8.6 (Pin_6), U10.B3 (PA15); no longer J4.6 (Pin_6)
- net PA1_SPI1_SCK: now also U10.G3 (PA1)
- net PA2_LPUART1_TX: now also U10.H2 (PA2)
- net PA3_LPUART1_RX: now also U10.H1 (PA3)
- net PA4_SPI1_NSS: now also U10.J1 (PA4)
- net PA5: now also J8.2 (Pin_2), U10.J2 (PA5); no longer J4.2 (Pin_2)
- net PA6_SPI1_MISO: now also U10.F4 (PA6)
- net PA7: now also J8.3 (Pin_3), U10.H3 (PA7); no longer J4.3 (Pin_3)
- net PA8_MCO: now also J8.4 (Pin_4), U10.J3 (PA8); no longer J4.4 (Pin_4)
- net PA9: now also J8.5 (Pin_5), U10.E5 (PA9); no longer J4.5 (Pin_5)
- net PB0: now also J8.7 (Pin_7), U10.F6 (PB0); no longer J4.7 (Pin_7)
- net PB1: now also J4.1 (Pin_1), U10.E7 (PB1)
- net PB10: now also J8.13 (Pin_13), U10.H4 (PB10)
- net PB11: now also J8.12 (Pin_12), U10.G4 (PB11)
- net PB12: now also J8.10 (Pin_10), U10.E6 (PB12); no longer J4.10 (Pin_10)
- net PB13: now also J4.11 (Pin_11), U10.D7 (PB13)
- net PB14: now also J4.10 (Pin_10), U10.C6 (PB14)
- net PB15: now also J4.12 (Pin_12), U10.B4 (PB15)
- net PB2: now also J8.8 (Pin_8), U10.D8 (PB2); no longer J4.8 (Pin_8)
- net PB3_SWO: now also U10.C1 (PB3)
- net PB4: now also J8.9 (Pin_9), U10.C2 (PB4); no longer J4.9 (Pin_9)
- net PB5_SPI1_MOSI: now also U10.D2 (PB5)
- net PB6_USART1_TX: now also U10.E1 (PB6)
- net PB7_I2C1_SDA: now also U10.C3 (PB7)
- net PB8_I2C1_SCL: now also U10.D3 (PB8)
- net PB9: now also J8.11 (Pin_11), U10.C4 (PB9)
- net PC0: now also J4.2 (Pin_2), U10.F2 (PC0)
- net PC1: now also J4.3 (Pin_3), U10.F1 (PC1)
- net PC13: now also U10.C7 (PC13)
- net PC14-OSC32_IN: now also R17.2, U10.B6 (PC14)
- net PC15-OSC32_OUT: now also J4.7 (Pin_7), U10.C5 (PC15); no longer J4.11 (Pin_11)
- net PC2: now also J4.4 (Pin_4), U10.D4 (PC2)
- net PC3: now also J4.5 (Pin_5), U10.D5 (PC3)
- net PC4: now also J4.6 (Pin_6), U10.F3 (PC4)
- net PC5: now also J4.8 (Pin_8), U10.E4 (PC5)
- net PC6: now also J4.9 (Pin_9), U10.G2 (PC6)
- net PH0-OSC_IN: now also U10.G9 (OSC_IN), Y4.3
- net PH1-OSC_OUT: now also U10.F8 (OSC_OUT), Y4.1
- net RFI_N: now also U10.H7 (RFI_N)
- net RFI_P: now also U10.J6 (RFI_P)
- net RFO_HP: now also U10.J9 (RFO_HP)
- net VBAT: now also U10.A8 (VBAT)
- net VFBSMPS: now also C63.1, C72.1, L9.1, U10.B2 (VFBSMPS), U10.F7 (VDDRF1V55)
- net VLXSMPS: now also L9.2, U10.B1 (VLXSMPS)
- net VR_PA: now also U10.H9 (VR_PA)
- new net: R17.1, Y5.3 (OUTPUT)
- no-connect marks 11 -> 9
Other:
- note removed: "Peripherals: 1. EEPROM memory chips (SPI or I2C) 2. Bluetooth 3. GPS 4. Orientation sensor (MEMS) 5. USB 6. Ethernet (Maybe) 7. A set of user buttons (maybe 4)"
- moved on the sheet: BH1, C16, C18, C19, C20, C21, C22, C23, C24, C25, C26, C27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

Commit message: Update
Parts:
- Y5: value Clock_ECS-327MVATX-7-CN-TR -> Clock_ECS-327MVATX-3-CN-TR
Changed lines of the file:
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@@
 			)
 		)
-		(property "Value" "Clock_ECS-327MVATX-7-CN-TR"
+		(property "Value" "Clock_ECS-327MVATX-3-CN-TR"
 			(at 217.424 203.962 0)
 			(effects
