File: LoRa_Board_STM32WL55JCI6.kicad_pcb (KiCad board)
At the start: 4 copper layers, 98 parts, among them J1 LPUART1_Headers, J10 Power Select Jumpers, J11 Debug_Pins, J13 SMA PCB END LAUNCH JACK ROUND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, J14 USB_B_Micro, J16 BOOT0_Jumper, J2 I2C1_Headers, J3 Power Pins, J4 Pin_Headers_2, J5 SPI1_Headers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

Commit message: Update
Routing:
- net /PC4: vias 0 -> 1
- net /PB11: vias 0 -> 1
- net /PA6_SPI1_MISO: vias 0 -> 1
- net /PA1_SPI1_SCK: vias 0 -> 1
Changed lines of the file:
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@@
 		(net 28)
+	)
+	(via
+		(at 97.3 70)
+		(size 0.3)
+		(drill 0.15)
+		(layers "F.Cu" "B.Cu")
+		(net 44)
+	)
+	(via
+		(at 97.8 70.5)
+		(size 0.3)
+		(drill 0.15)
+		(layers "F.Cu" "B.Cu")
+		(net 56)
 	)
 	(segment
@@
 		(net 77)
 	)
+	(via
+		(at 97.3 70.5)
+		(size 0.3)
+		(drill 0.15)
+		(layers "F.Cu" "B.Cu")
+		(net 83)
+	)
+	(via
+		(at 97.8 70)
+		(size 0.3)
+		(drill 0.15)
+		(layers "F.Cu" "B.Cu")
+		(net 85)
+	)
 	(segment

Commit message: Update
Routing:
- net /PC14-OSC32_IN: track 0.00 -> 2.79 mm
- net GND: track 11.9 -> 9.33 mm, vias 0 -> 2
- net /PA7: track 0.00 -> 2.07 mm
- net /PA8_MCO: track 0.00 -> 1.30 mm
- net +3.3VA: track 3.58 -> 2.33 mm
- net /PA5: track 0.00 -> 1.20 mm
- net /VFBSMPS: vias 0 -> 1
- net /PC4: vias 1 -> 0
- net /PB11: vias 1 -> 0
- net /PA6_SPI1_MISO: vias 1 -> 0
- net /PA1_SPI1_SCK: vias 1 -> 0
- net /NRST: vias 0 -> 1
Changed lines of the file:
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@@
 		(tags "BGA 73 0.5")
 		(property "Reference" "U10"
-			(at 0 -3.5 0)
+			(at -2 -4.2 0)
 			(layer "F.SilkS")
 			(effects
 				(font
 					(size 1 1)
-					(thickness 0.15)
+					(thickness 0.153)
 				)
 			)
@@
 	)
 	(segment
-		(start 99.3 67.99)
-		(end 98.96 67.65)
-		(width 0.1)
-		(layer "F.Cu")
-		(net 3)
-	)
-	(segment
 		(start 98.3 70.5)
 		(end 98.8 70.5)
@@
 	)
 	(segment
-		(start 98.96 67.65)
-		(end 98.96 65.53)
-		(width 0.1)
-		(layer "F.Cu")
-		(net 3)
-	)
-	(segment
 		(start 99.3 70.5)
 		(end 99.8 70.5)
@@
 		(net 3)
 	)
+	(via
+		(at 99.3 68)
+		(size 0.3)
+		(drill 0.2)
+		(layers "F.Cu" "B.Cu")
+		(net 3)
+	)
+	(via
+		(at 97.3 69.5)
+		(size 0.3)
+		(drill 0.2)
+		(layers "F.Cu" "B.Cu")
+		(net 3)
+	)
 	(segment
 		(start 99.8 65.19)
@@
 		(net 27)
 	)
+	(via
+		(at 99.3 70)
+		(size 0.3)
+		(drill 0.2)
+		(layers "F.Cu" "B.Cu")
+		(net 27)
+	)
 	(segment
 		(start 98.3 65.68)
@@
 	(segment
 		(start 98.3 68)
-		(end 98.66 67.64)
-		(width 0.1)
-		(layer "F.Cu")
-		(net 28)
-	)
-	(segment
-		(start 98.66 67.64)
-		(end 98.66 66.4)
-		(width 0.1)
+		(end 98.3 67.5)
+		(width 0.15)
 		(layer "F.Cu")
 		(net 28)
@@
 	)
 	(via
-		(at 97.3 70)
-		(size 0.3)
-		(drill 0.15)
-		(layers "F.Cu" "B.Cu")
-		(net 44)
-	)
-	(via
-		(at 97.8 70.5)
+		(at 98.3 70)
 		(size 0.3)
-		(drill 0.15)
+		(drill 0.2)
 		(layers "F.Cu" "B.Cu")
-		(net 56)
+		(net 29)
 	)
 	(segment
@@
 	)
 	(segment
+		(start 96.8 71.5)
+		(end 96.8 72.7)
+		(width 0.15)
+		(layer "F.Cu")
+		(net 60)
+	)
+	(segment
+		(start 97.3 71.5)
+		(end 97.3 72.8)
+		(width 0.15)
+		(layer "F.Cu")
+		(net 65)
+	)
+	(segment
 		(start 96.8 68.5)
 		(end 96.485 68.815)
@@
 	)
 	(segment
+		(start 97.6 71.3)
+		(end 97.6 72.8)
+		(width 0.15)
+		(layer "F.Cu")
+		(net 68)
+	)
+	(segment
+		(start 97.3 71)
+		(end 97.6 71.3)
+		(width 0.15)
+		(layer "F.Cu")
+		(net 68)
+	)
+	(segment
+		(start 97.6 72.8)
+		(end 97.7 72.9)
+		(width 0.15)
+		(layer "F.Cu")
+		(net 68)
+	)
+	(segment
 		(start 97.8 67.5)
 		(end 97.8 65.61)
@@
 		(net 77)
 	)
-	(via
-		(at 97.3 70.5)
-		(size 0.3)
-		(drill 0.15)
-		(layers "F.Cu" "B.Cu")
-		(net 83)
+	(segment
+		(start 98.96 67.84)
+		(end 98.96 65.36)
+		(width 0.15)
+		(layer "F.Cu")
+		(net 90)
 	)
-	(via
-		(at 97.8 70)
-		(size 0.3)
-		(drill 0.15)
-		(layers "F.Cu" "B.Cu")
-		(net 85)
+	(segment
+		(start 98.8 68)
+		(end 98.96 67.84)
+		(width 0.15)
+		(layer "F.Cu")
+		(net 90)
+	)
+	(segment
+		(start 98.96 65.36)
+		(end 98.9 65.3)
+		(width 0.15)
+		(layer "F.Cu")
+		(net 90)
 	)
 	(segment
